File: DontWorry.kicad_sch (KiCad schematic)
At the start: 25 parts, among them J1 Conn_02x03_Odd_Even, J2 Conn_02x03_Odd_Even, J3 Conn_01x14, Q5 BC849, Q6 BC849, Q7 BC849, Q8 BC849, Q9 BC849, U1 CC56-12YWA

Commit message: Updated PCB
Parts:
- removed J3: Conn_01x14, Connector_PinHeader_2.54mm:PinHeader_2x07_P2.54mm_Vertical, symbol Connector_Generic:Conn_01x14
- added J4: Conn_01x06, Connector_PinHeader_2.54mm:PinHeader_2x03_P2.54mm_Vertical, symbol Connector_Generic:Conn_01x06
- added R14, R15, R16, R17, R18: 10K, Resistor_SMD:R_0805_2012Metric, symbol Device:R_Small
Connections:
- net +5V: now also J2.1 (Pin_1), J2.2 (Pin_2), J2.3 (Pin_3), J2.4 (Pin_4), J2.5 (Pin_5), J2.6 (Pin_6), J4.2 (Pin_2)
- net A1: now also J1.1 (Pin_1), R14.1
- net A2: now also J1.3 (Pin_3), R15.1
- net A3: now also J1.5 (Pin_5), R16.1
- net A4: now also J1.2 (Pin_2), R18.1
- net A5: now also J1.4 (Pin_4), R17.1
- net GND: now also J4.1 (Pin_1), R14.2, R15.2, R16.2, R17.2, R18.2
- net RX: now also J4.5 (Pin_5)
- net SCL: now also J4.4 (Pin_4)
- net SDA: now also J4.3 (Pin_3)
- net TX: now also J4.6 (Pin_6)
- no-connect marks 4 -> 5
Other:
- note added: ""Bombenentschärfung" Kabelbrücken"
- note added: "I2C & UART"
- moved on the sheet: A1, BZ1, H4, J1, J2, Q5, Q6, Q7, Q8, Q9, R1, R10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
