File: DontWorry.kicad_pcb (KiCad board)
At the start: 2 copper layers, 71 x 54 mm, 30 parts, among them J1 Conn_02x03_Odd_Even, J2 Conn_02x03_Odd_Even, J4 Conn_01x06, Q5 BC849, Q6 BC849, Q7 BC849, Q8 BC849, Q9 BC849

Commit message: Moved Buzzer south for increased pin clearance
Parts:
- H4: renamed from H4 (GND)
- U1: renamed from 7-SEG DISPLAY CC
- moved BZ1 0.10 mm to (155.1, 60.8)
Changed lines of the file:
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@@
 		(descr "4 digit 7 segment green LED, http://www.kingbrightusa.com/images/catalog/SPEC/CC56-12YWA.pdf")
 		(tags "4 digit 7 segment green LED")
-		(property "Reference" "7-SEG DISPLAY CC"
+		(property "Reference" "U1"
 			(at 7.3952 34.11 90)
 			(layer "F.SilkS" knockout)
@@
 	(footprint "Buzzer_Beeper:Buzzer_12x9.5RM7.6"
 		(layer "F.Cu")
-		(at 155.1 60.7 -90)
+		(at 155.1 60.8 -90)
 		(descr "Generic Buzzer, D12mm height 9.5mm with RM7.6mm")
 		(tags "buzzer")
@@
 			(net 49 "unconnected-(J1-Pin_6-Pad6)")
 			(pinfunction "Pin_6")
-			(pintype "passive")
+			(pintype "passive+no_connect")
 		)
 		(model "${KICAD8_3DMODEL_DIR}/Connector_PinHeader_2.54mm.3dshapes/PinHeader_2x03_P2.54mm_Vertical.wrl"
@@
 		(descr "Mounting Hole 3.2mm, M3, DIN965")
 		(tags "mounting hole 3.2mm m3 din965")
-		(property "Reference" "H4 (GND)"
+		(property "Reference" "H4"
 			(at -0.1 -4.9 0)
 			(layer "F.SilkS" knockout)
@@
 			(net 6 "unconnected-(A1-~{RESET}-Pad3)")
 			(pinfunction "~{RESET}")
-			(pintype "input")
+			(pintype "input+no_connect")
 		)
 		(pad "4" thru_hole oval
